File: NodeMCU_Sensors/NodeMCU_Sensors.sch (KiCad schematic (older format))
At the start: 10 parts, among them J1 Conn_02x15_Odd_Even, J2 Conn_02x15_Odd_Even, J3 Conn_01x04, J4 Conn_01x04, J5 Conn_01x04, J6 Audio-Jack-3_2Switches, J7 Audio-Jack-3_2Switches, J8 Audio-Jack-3_2Switches, SW1 SW_Push

Commit message: Place parts according to layout plan
Parts:
- SW1: footprint Button_Switch_THT:SW_PUSH_6mm -> Button_Switch_THT:SW_Tactile_SPST_Angled_PTS645Vx39-2LFS
- renumbered J7 to 1wire1, J6 to 1wire2, J8 to Analog1, J4 to MPU6050, J3 to OLED1, J5 to SIL1
Changed lines of the file:
@@
 EESchema Schematic File Version 4
+LIBS:NodeMCU_Sensors-cache
 EELAYER 26 0
 EELAYER END
@@
 $EndComp
 $Comp
-L Connector_Generic:Conn_01x04 J3
+L Connector_Generic:Conn_01x04 OLED1
 U 1 1 5A69B21D
 P 3450 1450
-F 0 "J3" V 3416 1162 50  0000 R CNN
+F 0 "OLED1" V 3416 1162 50  0000 R CNN
 F 1 "Conn_01x04" V 3325 1162 50  0000 R CNN
 F 2 "Connector_PinSocket_2.54mm:PinSocket_1x04_P2.54mm_Vertical" H 3450 1450 50  0001 C CNN
@@
 $EndComp
 $Comp
-L Connector_Generic:Conn_01x04 J4
+L Connector_Generic:Conn_01x04 MPU6050
 U 1 1 5A69B28D
 P 3450 2100
-F 0 "J4" V 3416 1812 50  0000 R CNN
+F 0 "MPU6050" V 3416 1812 50  0000 R CNN
 F 1 "Conn_01x04" V 3325 1812 50  0000 R CNN
 F 2 "Connector_PinSocket_2.54mm:PinSocket_1x04_P2.54mm_Vertical" H 3450 2100 50  0001 C CNN
@@
 $EndComp
 $Comp
-L Connector_Specialized:Audio-Jack-3_2Switches J6
+L Connector_Specialized:Audio-Jack-3_2Switches 1wire2
 U 1 1 5A69B495
 P 5650 1650
-F 0 "J6" H 5626 2075 50  0000 C CNN
+F 0 "1wire2" H 5626 2075 50  0000 C CNN
 F 1 "Audio-Jack-3_2Switches" H 5626 1984 50  0000 C CNN
 F 2 "Connector_Audio:Jack_3.5mm_PJ320E_Horizontal" H 5900 1750 50  0001 C CNN
@@
 $EndComp
 $Comp
-L Connector_Specialized:Audio-Jack-3_2Switches J7
+L Connector_Specialized:Audio-Jack-3_2Switches 1wire1
 U 1 1 5A69B507
 P 5650 2450
-F 0 "J7" H 5626 2875 50  0000 C CNN
+F 0 "1wire1" H 5626 2875 50  0000 C CNN
 F 1 "Audio-Jack-3_2Switches" H 5626 2784 50  0000 C CNN
 F 2 "Connector_Audio:Jack_3.5mm_PJ320E_Horizontal" H 5900 2550 50  0001 C CNN
@@
 $EndComp
 $Comp
-L Connector_Specialized:Audio-Jack-3_2Switches J8
+L Connector_Specialized:Audio-Jack-3_2Switches Analog1
 U 1 1 5A69B5CA
 P 5650 3250
-F 0 "J8" H 5626 3675 50  0000 C CNN
+F 0 "Analog1" H 5626 3675 50  0000 C CNN
 F 1 "Audio-Jack-3_2Switches" H 5626 3584 50  0000 C CNN
 F 2 "Connector_Audio:Jack_3.5mm_PJ320E_Horizontal" H 5900 3350 50  0001 C CNN
@@
 $EndComp
 $Comp
-L Connector_Generic:Conn_01x04 J5
+L Connector_Generic:Conn_01x04 SIL1
 U 1 1 5A69B67B
 P 3450 2800
-F 0 "J5" V 3416 2512 50  0000 R CNN
+F 0 "SIL1" V 3416 2512 50  0000 R CNN
 F 1 "Conn_01x04" V 3325 2512 50  0000 R CNN
 F 2 "Connector_PinSocket_2.54mm:PinSocket_1x04_P2.54mm_Vertical" H 3450 2800 50  0001 C CNN
@@
 F 0 "SW1" H 7850 1785 50  0000 C CNN
 F 1 "SW_Push" H 7850 1694 50  0000 C CNN
-F 2 "Button_Switch_THT:SW_PUSH_6mm" H 7850 1700 50  0001 C CNN
+F 2 "Button_Switch_THT:SW_Tactile_SPST_Angled_PTS645Vx39-2LFS" H 7850 1700 50  0001 C CNN
 F 3 "" H 7850 1700 50  0001 C CNN
 	1    7850 1500

Commit message: Wire up i2c sensors
Parts:
- J1, J2: footprint Connector_PinSocket_2.54mm:PinSocket_2x15_P2.54mm_Vertical -> Socket_Strips:Socket_Strip_Straight_2x15_Pitch2.54mm
- MPU6050, OLED1: footprint Connector_PinSocket_2.54mm:PinSocket_1x04_P2.54mm_Vertical -> Socket_Strips:Socket_Strip_Straight_1x04_Pitch2.54mm
- SHT21: renamed from SIL1; footprint Connector_PinSocket_2.54mm:PinSocket_1x04_P2.54mm_Vertical -> Socket_Strips:Socket_Strip_Straight_1x04_Pitch2.54mm
Other:
- note added: "D1 - SCL\nD2 - SDA"
- note added: "i2c bus devices with 4-pin headers"
Changed lines of the file:
@@
 F 0 "J1" H 1750 3067 50  0000 C CNN
 F 1 "Conn_02x15_Odd_Even" H 1750 2976 50  0000 C CNN
-F 2 "Connector_PinSocket_2.54mm:PinSocket_2x15_P2.54mm_Vertical" H 1700 2150 50  0001 C CNN
+F 2 "Socket_Strips:Socket_Strip_Straight_2x15_Pitch2.54mm" H 1700 2150 50  0001 C CNN
 F 3 "~" H 1700 2150 50  0001 C CNN
 	1    1700 2150
@@
 F 0 "J2" H 1750 4867 50  0000 C CNN
 F 1 "Conn_02x15_Odd_Even" H 1750 4776 50  0000 C CNN
-F 2 "Connector_PinSocket_2.54mm:PinSocket_2x15_P2.54mm_Vertical" H 1700 3950 50  0001 C CNN
+F 2 "Socket_Strips:Socket_Strip_Straight_2x15_Pitch2.54mm" H 1700 3950 50  0001 C CNN
 F 3 "~" H 1700 3950 50  0001 C CNN
 	1    1700 3950
@@
 F 0 "OLED1" V 3416 1162 50  0000 R CNN
 F 1 "Conn_01x04" V 3325 1162 50  0000 R CNN
-F 2 "Connector_PinSocket_2.54mm:PinSocket_1x04_P2.54mm_Vertical" H 3450 1450 50  0001 C CNN
+F 2 "Socket_Strips:Socket_Strip_Straight_1x04_Pitch2.54mm" H 3450 1450 50  0001 C CNN
 F 3 "~" H 3450 1450 50  0001 C CNN
 	1    3450 1450
@@
 L Connector_Generic:Conn_01x04 MPU6050
 U 1 1 5A69B28D
-P 3450 2100
-F 0 "MPU6050" V 3416 1812 50  0000 R CNN
-F 1 "Conn_01x04" V 3325 1812 50  0000 R CNN
-F 2 "Connector_PinSocket_2.54mm:PinSocket_1x04_P2.54mm_Vertical" H 3450 2100 50  0001 C CNN
-F 3 "~" H 3450 2100 50  0001 C CNN
-	1    3450 2100
-	0    -1   -1   0
+P 3550 2400
+F 0 "MPU6050" V 3516 2112 50  0000 R CNN
+F 1 "Conn_01x04" V 3425 2112 50  0000 R CNN
+F 2 "Socket_Strips:Socket_Strip_Straight_1x04_Pitch2.54mm" H 3550 2400 50  0001 C CNN
+F 3 "~" H 3550 2400 50  0001 C CNN
+	1    3550 2400
+	0    1    1    0
 $EndComp
 $Comp
@@
 $EndComp
 $Comp
-L Connector_Generic:Conn_01x04 SIL1
+L Connector_Generic:Conn_01x04 SHT21
 U 1 1 5A69B67B
-P 3450 2800
-F 0 "SIL1" V 3416 2512 50  0000 R CNN
-F 1 "Conn_01x04" V 3325 2512 50  0000 R CNN
-F 2 "Connector_PinSocket_2.54mm:PinSocket_1x04_P2.54mm_Vertical" H 3450 2800 50  0001 C CNN
-F 3 "~" H 3450 2800 50  0001 C CNN
-	1    3450 2800
-	0    -1   -1   0
+P 3600 3050
+F 0 "SHT21" V 3566 2762 50  0000 R CNN
+F 1 "Conn_01x04" V 3475 2762 50  0000 R CNN
+F 2 "Socket_Strips:Socket_Strip_Straight_1x04_Pitch2.54mm" H 3600 3050 50  0001 C CNN
+F 3 "~" H 3600 3050 50  0001 C CNN
+	1    3600 3050
+	0    1    1    0
 $EndComp
 $Comp
@@
 Text GLabel 2000 3250 2    50   Input ~ 0
 D0
+Text Notes 3300 1100 0    50   ~ 0
+D1 - SCL\nD2 - SDA
+Text GLabel 3350 1650 3    50   Input ~ 0
+3V3
+Text GLabel 3450 1650 3    50   Input ~ 0
+GND
+Text GLabel 3550 1650 3    50   Input ~ 0
+D1
+Text GLabel 3650 1650 3    50   Input ~ 0
+D2
+Text Notes 2900 850  0    50   ~ 0
+i2c bus devices with 4-pin headers
+Text GLabel 3350 2200 1    50   Input ~ 0
+3V3
+Text GLabel 3450 2200 1    50   Input ~ 0
+GND
+Text GLabel 3550 2200 1    50   Input ~ 0
+D1
+Text GLabel 3650 2200 1    50   Input ~ 0
+D2
+Text GLabel 3400 2850 1    50   Input ~ 0
+3V3
+Text GLabel 3500 2850 1    50   Input ~ 0
+GND
+Text GLabel 3600 2850 1    50   Input ~ 0
+D1
+Text GLabel 3700 2850 1    50   Input ~ 0
+D2
 $EndSCHEMATC

Commit message: Route 3.5mm jacks
Parts:
- 1wire1, Analog1: symbol Connector_Specialized:Audio-Jack-3_2Switches -> Connector_Specialized:Audio-Jack-3
- 1wire2: symbol Connector_Specialized:Audio-Jack-3_2Switches -> Connector_Specialized:Audio-Jack-3; manf# (none) -> PJ320E
Other:
- note added: "1-wire protocol with programmable pinout"
- note added: "Analog input (max 1V without divider)"
Changed lines of the file:
@@
 $EndComp
 $Comp
-L Connector_Specialized:Audio-Jack-3_2Switches 1wire2
+L Connector_Specialized:Audio-Jack-3 1wire2
 U 1 1 5A69B495
 P 5650 1650
@@
 F 2 "Connector_Audio:Jack_3.5mm_PJ320E_Horizontal" H 5900 1750 50  0001 C CNN
 F 3 "~" H 5900 1750 50  0001 C CNN
+F 4 "PJ320E" H 5650 1650 50  0001 C CNN "manf#"
 	1    5650 1650
 	1    0    0    -1
 $EndComp
 $Comp
-L Connector_Specialized:Audio-Jack-3_2Switches 1wire1
+L Connector_Specialized:Audio-Jack-3 1wire1
 U 1 1 5A69B507
 P 5650 2450
@@
 $EndComp
 $Comp
-L Connector_Specialized:Audio-Jack-3_2Switches Analog1
+L Connector_Specialized:Audio-Jack-3 Analog1
 U 1 1 5A69B5CA
 P 5650 3250
@@
 L pspice:R R1
 U 1 1 5A69BB4C
-P 6600 2800
-F 0 "R1" H 6668 2846 50  0000 L CNN
-F 1 "R" H 6668 2755 50  0000 L CNN
-F 2 "Resistor_THT:R_Axial_DIN0204_L3.6mm_D1.6mm_P5.08mm_Horizontal" H 6600 2800 50  0001 C CNN
-F 3 "" H 6600 2800 50  0001 C CNN
-	1    6600 2800
+P 6550 2000
+F 0 "R1" H 6618 2046 50  0000 L CNN
+F 1 "R" H 6618 1955 50  0000 L CNN
+F 2 "Resistor_THT:R_Axial_DIN0204_L3.6mm_D1.6mm_P5.08mm_Horizontal" H 6550 2000 50  0001 C CNN
+F 3 "" H 6550 2000 50  0001 C CNN
+	1    6550 2000
 	1    0    0    -1
 $EndComp
@@
 Text GLabel 3700 2850 1    50   Input ~ 0
 D2
+Text GLabel 5450 3350 3    50   Input ~ 0
+GND
+Text GLabel 5850 3250 2    50   Input ~ 0
+A0
+Text GLabel 5850 2350 2    50   Input ~ 0
+D6
+Text GLabel 5450 2550 3    50   Input ~ 0
+D8
+Text GLabel 5850 2450 2    50   Input ~ 0
+D7
+Text GLabel 5850 1550 2    50   Input ~ 0
+D6
+Text GLabel 5850 1650 2    50   Input ~ 0
+D7
+Text GLabel 5450 1750 3    50   Input ~ 0
+D8
+Text Notes 4950 3700 0    50   ~ 0
+Analog input (max 1V without divider)
+Text Notes 5000 1050 0    50   ~ 0
+1-wire protocol with programmable pinout
+Text GLabel 8050 1500 2    50   Input ~ 0
+D5
+Text GLabel 7650 1500 0    50   Input ~ 0
+GND
 $EndSCHEMATC

Commit message: Basic autorouted board
Parts:
- added R2: 39K, Resistors_THT:R_Axial_DIN0204_L3.6mm_D1.6mm_P5.08mm_Horizontal, symbol Device:R
- added R3: 10K, Resistors_THT:R_Axial_DIN0204_L3.6mm_D1.6mm_P5.08mm_Horizontal, symbol Device:R
- R1: value R -> 4.7K
Connections:
- wire segments 30 -> 34
Changed lines of the file:
@@
 P 6550 2000
 F 0 "R1" H 6618 2046 50  0000 L CNN
-F 1 "R" H 6618 1955 50  0000 L CNN
+F 1 "4.7K" H 6618 1955 50  0000 L CNN
 F 2 "Resistor_THT:R_Axial_DIN0204_L3.6mm_D1.6mm_P5.08mm_Horizontal" H 6550 2000 50  0001 C CNN
 F 3 "" H 6550 2000 50  0001 C CNN
@@
 Text GLabel 5450 3350 3    50   Input ~ 0
 GND
-Text GLabel 5850 3250 2    50   Input ~ 0
-A0
 Text GLabel 5850 2350 2    50   Input ~ 0
 D6
 Text GLabel 5450 2550 3    50   Input ~ 0
-D8
+GND
 Text GLabel 5850 2450 2    50   Input ~ 0
 D7
@@
 D7
 Text GLabel 5450 1750 3    50   Input ~ 0
-D8
+GND
 Text Notes 4950 3700 0    50   ~ 0
 Analog input (max 1V without divider)
@@
 Text GLabel 7650 1500 0    50   Input ~ 0
 GND
+Text GLabel 6550 1750 1    50   Input ~ 0
+D6
+Text GLabel 6550 2250 3    50   Input ~ 0
+D7
+$Comp
+L Device:R R3
+U 1 1 5A6DB795
+P 6300 3450
+F 0 "R3" V 6093 3450 50  0000 C CNN
+F 1 "10K" V 6184 3450 50  0000 C CNN
+F 2 "Resistors_THT:R_Axial_DIN0204_L3.6mm_D1.6mm_P5.08mm_Horizontal" V 6230 3450 50  0001 C CNN
+F 3 "" H 6300 3450 50  0001 C CNN
+	1    6300 3450
+	0    1    1    0
+$EndComp
+$Comp
+L Device:R R2
+U 1 1 5A6DB7DB
+P 5950 3450
+F 0 "R2" V 5743 3450 50  0000 C CNN
+F 1 "39K" V 5834 3450 50  0000 C CNN
+F 2 "Resistors_THT:R_Axial_DIN0204_L3.6mm_D1.6mm_P5.08mm_Horizontal" V 5880 3450 50  0001 C CNN
+F 3 "" H 5950 3450 50  0001 C CNN
+	1    5950 3450
+	0    1    1    0
+$EndComp
+Text GLabel 6450 3450 2    50   Input ~ 0
+GND
+Wire Wire Line
+	6100 3450 6150 3450
+Wire Wire Line
+	5800 3450 5800 3300
+Wire Wire Line
+	5800 3300 5850 3300
+Wire Wire Line
+	5850 3300 5850 3250
+Text GLabel 6100 3450 1    50   Input ~ 0
+A0
 $EndSCHEMATC

Commit message: Add 3V3 supply to analog pin and re-route
Parts:
- R2: value 39K -> 23.2K
Connections:
- wire segments 34 -> 31
Other:
- note added: "Analog input (max 3.3V with divider)"
- note removed: "Analog input (max 1V without divider)"
Changed lines of the file:
@@
 GND
 Text Notes 4950 3700 0    50   ~ 0
-Analog input (max 1V without divider)
+Analog input (max 3.3V with divider)
 Text Notes 5000 1050 0    50   ~ 0
 1-wire protocol with programmable pinout
@@
 L Device:R R3
 U 1 1 5A6DB795
-P 6300 3450
-F 0 "R3" V 6093 3450 50  0000 C CNN
-F 1 "10K" V 6184 3450 50  0000 C CNN
-F 2 "Resistors_THT:R_Axial_DIN0204_L3.6mm_D1.6mm_P5.08mm_Horizontal" V 6230 3450 50  0001 C CNN
-F 3 "" H 6300 3450 50  0001 C CNN
-	1    6300 3450
+P 6350 3150
+F 0 "R3" V 6143 3150 50  0000 C CNN
+F 1 "10K" V 6234 3150 50  0000 C CNN
+F 2 "Resistors_THT:R_Axial_DIN0204_L3.6mm_D1.6mm_P5.08mm_Horizontal" V 6280 3150 50  0001 C CNN
+F 3 "" H 6350 3150 50  0001 C CNN
+	1    6350 3150
 	0    1    1    0
 $EndComp
@@
 L Device:R R2
 U 1 1 5A6DB7DB
-P 5950 3450
-F 0 "R2" V 5743 3450 50  0000 C CNN
-F 1 "39K" V 5834 3450 50  0000 C CNN
-F 2 "Resistors_THT:R_Axial_DIN0204_L3.6mm_D1.6mm_P5.08mm_Horizontal" V 5880 3450 50  0001 C CNN
-F 3 "" H 5950 3450 50  0001 C CNN
-	1    5950 3450
+P 6000 3150
+F 0 "R2" V 5793 3150 50  0000 C CNN
+F 1 "23.2K" V 5884 3150 50  0000 C CNN
+F 2 "Resistors_THT:R_Axial_DIN0204_L3.6mm_D1.6mm_P5.08mm_Horizontal" V 5930 3150 50  0001 C CNN
+F 3 "" H 6000 3150 50  0001 C CNN
+	1    6000 3150
 	0    1    1    0
 $EndComp
-Text GLabel 6450 3450 2    50   Input ~ 0
+Text GLabel 6500 3150 2    50   Input ~ 0
 GND
 Wire Wire Line
-	6100 3450 6150 3450
-Wire Wire Line
-	5800 3450 5800 3300
-Wire Wire Line
-	5800 3300 5850 3300
-Wire Wire Line
-	5850 3300 5850 3250
-Text GLabel 6100 3450 1    50   Input ~ 0
+	6150 3150 6200 3150
+Text GLabel 6150 3150 1    50   Input ~ 0
 A0
+Text GLabel 5850 3250 2    50   Input ~ 0
+3V3
 $EndSCHEMATC

Commit message: Adde makesmart logo
Parts:
- added G1: LOGO, project_footprints:makeSmart_logo, symbol makeSmart_logo:LOGO
- added G2: Logo_Open_Hardware_Small, Symbols:OSHW-Logo2_7.3x6mm_SilkScreen, symbol Graphic:Logo_Open_Hardware_Small
Changed lines of the file:
@@
 Text GLabel 5850 3250 2    50   Input ~ 0
 3V3
+$Comp
+L makeSmart_logo:LOGO G1
+U 1 1 5A705986
+P 7300 3850
+F 0 "G1" H 7300 3794 60  0001 C CNN
+F 1 "LOGO" H 7300 3906 60  0001 C CNN
+F 2 "project_footprints:makeSmart_logo" H 7300 3850 50  0001 C CNN
+F 3 "" H 7300 3850 50  0001 C CNN
+	1    7300 3850
+	1    0    0    -1
+$EndComp
+$Comp
+L Graphic:Logo_Open_Hardware_Small G2
+U 1 1 5A7068A1
+P 8250 3900
+F 0 "G2" H 8250 4175 50  0001 C CNN
+F 1 "Logo_Open_Hardware_Small" H 8250 3675 50  0001 C CNN
+F 2 "Symbols:OSHW-Logo2_7.3x6mm_SilkScreen" H 8250 3900 50  0001 C CNN
+F 3 "~" H 8250 3900 50  0001 C CNN
+	1    8250 3900
+	1    0    0    -1
+$EndComp
 $EndSCHEMATC

Commit message: Address #1 for V2 board
Parts:
- removed R2: 23.2K, Resistors_THT:R_Axial_DIN0204_L3.6mm_D1.6mm_P5.08mm_Horizontal, symbol Device:R
- removed R3: 10K, Resistors_THT:R_Axial_DIN0204_L3.6mm_D1.6mm_P5.08mm_Horizontal, symbol Device:R
- R1: footprint Resistor_THT:R_Axial_DIN0204_L3.6mm_D1.6mm_P5.08mm_Horizontal -> Resistors_SMD:R_0603_HandSoldering
- Temperature1: renamed from SHT21; manf# (none) -> (none)
Connections:
- wire segments 31 -> 30
Changed lines of the file:
@@
 $EndComp
 $Comp
-L Connector_Generic:Conn_01x04 SHT21
+L Connector_Generic:Conn_01x04 Temperature1
 U 1 1 5A69B67B
 P 3600 3050
-F 0 "SHT21" V 3566 2762 50  0000 R CNN
+F 0 "Temperature1" V 3566 2762 50  0000 R CNN
 F 1 "Conn_01x04" V 3475 2762 50  0000 R CNN
 F 2 "Socket_Strips:Socket_Strip_Straight_1x04_Pitch2.54mm" H 3600 3050 50  0001 C CNN
 F 3 "~" H 3600 3050 50  0001 C CNN
+F 4 " " H 3600 3050 50  0001 C CNN "manf#"
 	1    3600 3050
 	0    1    1    0
@@
 F 0 "R1" H 6618 2046 50  0000 L CNN
 F 1 "4.7K" H 6618 1955 50  0000 L CNN
-F 2 "Resistor_THT:R_Axial_DIN0204_L3.6mm_D1.6mm_P5.08mm_Horizontal" H 6550 2000 50  0001 C CNN
+F 2 "Resistors_SMD:R_0603_HandSoldering" H 6550 2000 50  0001 C CNN
 F 3 "" H 6550 2000 50  0001 C CNN
 	1    6550 2000
@@
 Text GLabel 3700 2850 1    50   Input ~ 0
 D2
-Text GLabel 5450 3350 3    50   Input ~ 0
-GND
 Text GLabel 5850 2350 2    50   Input ~ 0
 D6
@@
 Text GLabel 6550 2250 3    50   Input ~ 0
 D7
-$Comp
-L Device:R R3
-U 1 1 5A6DB795
-P 6350 3150
-F 0 "R3" V 6143 3150 50  0000 C CNN
-F 1 "10K" V 6234 3150 50  0000 C CNN
-F 2 "Resistors_THT:R_Axial_DIN0204_L3.6mm_D1.6mm_P5.08mm_Horizontal" V 6280 3150 50  0001 C CNN
-F 3 "" H 6350 3150 50  0001 C CNN
-	1    6350 3150
-	0    1    1    0
-$EndComp
-$Comp
-L Device:R R2
-U 1 1 5A6DB7DB
-P 6000 3150
-F 0 "R2" V 5793 3150 50  0000 C CNN
-F 1 "23.2K" V 5884 3150 50  0000 C CNN
-F 2 "Resistors_THT:R_Axial_DIN0204_L3.6mm_D1.6mm_P5.08mm_Horizontal" V 5930 3150 50  0001 C CNN
-F 3 "" H 6000 3150 50  0001 C CNN
-	1    6000 3150
-	0    1    1    0
-$EndComp
-Text GLabel 6500 3150 2    50   Input ~ 0
-GND
-Wire Wire Line
-	6150 3150 6200 3150
-Text GLabel 6150 3150 1    50   Input ~ 0
+Text GLabel 5850 3150 2    50   Input ~ 0
 A0
 Text GLabel 5850 3250 2    50   Input ~ 0
